File: hardware/flight_pcb/hab1_flight.kicad_sch (KiCad schematic)
At the start: 56 parts, among them J1 BATTERY 4xL91, J10 OLED SSD1306 (bench), J2 POWER SWITCH (on the box), J3 STDC14 SWD+VCP, J4 SPI FLASH module, J5 IMU GY-601N1, J6 BAROMETER BMP390, J7 GPS MAX-M10S, J8 DS18B20 probe, J9 LoRa E22-400M22S (adapter), Q1 AO3401A, SW1 RESET, U1 STM32G474RET6, U2 MIC5219-3.3

Commit message: hardware: generated starting PCB for the flight board (placed, not routed)
gen_pcb.py (run with KiCad's Python) builds hab1_flight.kicad_pcb from
the schematic netlist: CubeSat 1U outline 95.89 x 90.17 mm, 4 copper
layers, JLCPCB-friendly minimum rules, all 56 footprints from the KiCad
library with their nets and linked to the schematic symbols, placed in
zones (power top-left, MCU centre with decoupling around it, STDC14 and
reset at the bottom edge, GPS top edge, LoRa right edge, IMU/barometer/
flash sockets on the left, DS18B20 connector at the bottom edge, test
points bottom-right), GND plane on In1 and +3V3 plane on In2, module
body outlines on User.Drawings. It refuses to overwrite a board that
already has tracks.

Checks: ERC 0, netlist 0 mismatches, DRC schematic parity 0; remaining
DRC items are the unrouted connections and silkscreen cosmetics.
Schematic: mounting holes and test points excluded from the BOM,
per-part notes stay as sheet text only.

Co-Authored-By: Claude Opus 5.5 (1M context) <noreply@anthropic.com>
Claude-Session: https://claude.ai/code/session_01Y9WTd2yaDzj6r4py6E8uJo
Parts:
- H1, H2, H3, H4, TP1, TP10, TP2, TP3, TP4, TP5, TP6, TP7, TP8, TP9: now left out of the parts list
- J10: Note CONFIRM order GND VCC SCL SDA -> (none)
- J3: Note pin 13 VCP_RX (probe input) <- MCU TX; pin 14 VCP_TX -> MCU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 -> (none)
- J4: Note order DI CLK GND DO CS 3V3 as on the bench module -> (none)
- J5: Note order VCC GND SCLK SDI SDO CS INT1 INT2 as on the GY-601N1 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 -> (none)
- J6: Note CONFIRM order: VCC GND SCK SDI SDO(=high, addr 0x77) CSB(=h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 -> (none)
- J7: Note CONFIRM order: VCC GND TX(module) RX(module) -> (none)
- J8: Note red / yellow / black -> (none)
- J9: Note rev A: E22 on a header until HW-6 is done -> (none)
- Q1: Note reverse-polarity protection: body diode drain->source -> (none)
- U2: Note provisional, decide after HW-21 -> (none)
Changed lines of the file:
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@@
 			)
 		)
-		(property "Note" "reverse-polarity protection: body diode drain->source"
-			(at 251.46 121.92 0)
-			(effects
-				(font
-					(size 1.27 1.27)
-				)
-				(hide yes)
-			)
-		)
 		(pin "1"
 		)
@@
 			)
 		)
-		(property "Note" "provisional, decide after HW-21"
-			(at 251.46 170.18 0)
-			(effects
-				(font
-					(size 1.27 1.27)
-				)
-				(hide yes)
-			)
-		)
 		(pin "1"
 		)
@@
 			)
 		)
-		(property "Note" "pin 13 VCP_RX (probe input) <- MCU TX; pin 14 VCP_TX -> MCU RX"
-			(at 332.74 104.14 0)
-			(effects
-				(font
-					(size 1.27 1.27)
-				)
-				(hide yes)
-			)
-		)
 		(pin "1"
 		)
@@
 			)
 		)
-		(property "Note" "order DI CLK GND DO CS 3V3 as on the bench module"
-			(at 332.74 401.32 0)
-			(effects
-				(font
-					(size 1.27 1.27)
-				)
-				(hide yes)
-			)
-		)
 		(pin "1"
 		)
@@
 			)
 		)
-		(property "Note" "order VCC GND SCLK SDI SDO CS INT1 INT2 as on the GY-601N1 silkscreen"
-			(at 332.74 436.88 0)
-			(effects
-				(font
-					(size 1.27 1.27)
-				)
-				(hide yes)
-			)
-		)
 		(pin "1"
 		)
@@
 			)
 		)
-		(property "Note" "CONFIRM order: VCC GND SCK SDI SDO(=high, addr 0x77) CSB(=high, I2C)"
-			(at 332.74 472.44 0)
-			(effects
-				(font
-					(size 1.27 1.27)
-				)
-				(hide yes)
-			)
-		)
 		(pin "1"
 		)
@@
 			)
 		)
-		(property "Note" "CONFIRM order: VCC GND TX(module) RX(module)"
-			(at 332.74 500.38 0)
-			(effects
-				(font
-					(size 1.27 1.27)
-				)
-				(hide yes)
-			)
-		)
 		(pin "1"
 		)
@@
 			)
 		)
-		(property "Note" "red / yellow / black"
-			(at 332.74 528.32 0)
-			(effects
-				(font
-					(size 1.27 1.27)
-				)
-				(hide yes)
-			)
-		)
 		(pin "1"
 		)
@@
 			)
 		)
-		(property "Note" "rev A: E22 on a header until HW-6 is done"
-			(at 411.48 78.74 0)
-			(effects
-				(font
-					(size 1.27 1.27)
-				)
-				(hide yes)
-			)
-		)
 		(pin "1"
 		)
@@
 			)
 		)
-		(property "Note" "CONFIRM order GND VCC SCL SDA"
-			(at 411.48 137.16 0)
-			(effects
-				(font
-					(size 1.27 1.27)
-				)
-				(hide yes)
-			)
-		)
 		(pin "1"
 		)
@@
 		(unit 1)
 		(exclude_from_sim no)
-		(in_bom yes)
+		(in_bom no)
 		(on_board yes)
 		(dnp no)
@@
 		(unit 1)
 		(exclude_from_sim no)
-		(in_bom yes)
+		(in_bom no)
 		(on_board yes)
 		(dnp no)
@@
 		(unit 1)
 		(exclude_from_sim no)
-		(in_bom yes)
+		(in_bom no)
 		(on_board yes)
 		(dnp no)
@@
 		(unit 1)
 		(exclude_from_sim no)
-		(in_bom yes)
+		(in_bom no)
 		(on_board yes)
 		(dnp no)
@@
 		(unit 1)
 		(exclude_from_sim no)
-		(in_bom yes)
+		(in_bom no)
 		(on_board yes)
 		(dnp no)
@@
 		(unit 1)
 		(exclude_from_sim no)
-		(in_bom yes)
+		(in_bom no)
 		(on_board yes)
 		(dnp no)
@@
 		(unit 1)
 		(exclude_from_sim no)
-		(in_bom yes)
+		(in_bom no)
 		(on_board yes)
 		(dnp no)
@@
 		(unit 1)
 		(exclude_from_sim no)
-		(in_bom yes)
+		(in_bom no)
 		(on_board yes)
 		(dnp no)
@@
 		(unit 1)
 		(exclude_from_sim no)
-		(in_bom yes)
+		(in_bom no)
 		(on_board yes)
 		(dnp no)
@@
 		(unit 1)
 		(exclude_from_sim no)
-		(in_bom yes)
+		(in_bom no)
 		(on_board yes)
 		(dnp no)
@@
 		(unit 1)
 		(exclude_from_sim no)
-		(in_bom yes)
+		(in_bom no)
 		(on_board yes)
 		(dnp no)
@@
 		(unit 1)
 		(exclude_from_sim no)
-		(in_bom yes)
+		(in_bom no)
 		(on_board yes)
 		(dnp no)
@@
 		(unit 1)
 		(exclude_from_sim no)
-		(in_bom yes)
+		(in_bom no)
 		(on_board yes)
 		(dnp no)
@@
 		(unit 1)
 		(exclude_from_sim no)
-		(in_bom yes)
+		(in_bom no)
 		(on_board yes)
 		(dnp no)

Commit message: hardware: barometer and GPS sockets from the real module pinouts (HW-24)
BMP390 module has 7 pins: INT CS SDO SDI SCK VCC GND (was 6 guessed).
MAX-M10S module has 5 pins: VCC GND TX RX PPS (was 4); PPS goes to PA8
(TIM1_CH1) for precise time. ERC 0, netlist check 0 mismatches, PCB
schematic parity 0; 121 unrouted connections as expected.

Co-Authored-By: Claude Opus 5.5 (1M context) <noreply@anthropic.com>
Claude-Session: https://claude.ai/code/session_01Y9WTd2yaDzj6r4py6E8uJo
Parts:
- J6: footprint Connector_PinSocket_2.54mm:PinSocket_1x06_P2.54mm_Vertical -> Connector_PinSocket_2.54mm:PinSocket_1x07_P2.54mm_Vertical; symbol Connector_Generic:Conn_01x06 -> Connector_Generic:Conn_01x07
- J7: footprint Connector_PinSocket_2.54mm:PinSocket_1x04_P2.54mm_Vertical -> Connector_PinSocket_2.54mm:PinSocket_1x05_P2.54mm_Vertical; symbol Connector_Generic:Conn_01x04 -> Connector_Generic:Conn_01x05
Connections:
- net +3V3: now also J6.2 (Pin_2), J6.3 (Pin_3); no longer J6.1 (Pin_1), J6.5 (Pin_5)
- net GND: now also J6.7 (Pin_7); no longer J6.2 (Pin_2)
- net I2C_SCL: now also J6.5 (Pin_5); no longer J6.3 (Pin_3)
- net GPS_PPS: now reaches U1.42 (PA8)
- net GPS_PPS: now also J7.5 (Pin_5)
Other:
- note added: "order INT CS SDO SDI SCK VCC GND as on the module (checked 2026-09-29); CS high = I2C, SDO high = addr 0x77"
- note added: "order VCC GND TX RX PPS as on the module (checked 2026-09-29); module TX -> MCU RX"
- note removed: "CONFIRM order: VCC GND SCK SDI SDO(=high, addr 0x77) CSB(=high, I2C)"
- note removed: "CONFIRM order: VCC GND TX(module) RX(module)"
- moved on the sheet: J8
Changed lines of the file:
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@@
 		)
 	)
-	(no_connect
-		(at 147.32 129.54)
+	(label "GPS_PPS"
+		(at 147.32 129.54 0)
+		(fields_autoplaced yes)
+		(effects
+			(font
+				(size 1.27 1.27)
+			)
+			(justify left bottom)
+		)
 	)
 	(no_connect
@@
 	)
 	(symbol
-		(lib_id "Connector_Generic:Conn_01x06")
+		(lib_id "Connector_Generic:Conn_01x07")
 		(at 332.74 472.44 0)
 		(unit 1)
@@
 		(dnp no)
 		(property "Reference" "J6"
-			(at 331.47 463.55 0)
+			(at 331.47 461.01 0)
 			(effects
 				(font
@@
 			)
 		)
-		(property "Footprint" "Connector_PinSocket_2.54mm:PinSocket_1x06_P2.54mm_Vertical"
+		(property "Footprint" "Connector_PinSocket_2.54mm:PinSocket_1x07_P2.54mm_Vertical"
 			(at 332.74 472.44 0)
 			(effects
@@
 		(pin "6"
 		)
+		(pin "7"
+		)
 		(instances
 			(project "hab1_flight"
@@
 		)
 	)
+	(no_connect
+		(at 327.66 464.82)
+	)
 	(symbol
 		(lib_id "power:+3V3")
@@
 	)
 	(symbol
-		(lib_id "power:GND")
-		(at 327.66 469.9 270)
+		(lib_id "power:+3V3")
+		(at 327.66 469.9 90)
 		(unit 1)
 		(exclude_from_sim no)
@@
 			)
 		)
-		(property "Value" "GND"
+		(property "Value" "+3V3"
 			(at 330.2 474.98 0)
 			(effects
@@
 		)
 	)
-	(label "I2C_SCL"
+	(label "I2C_SDA"
 		(at 327.66 472.44 180)
 		(fields_autoplaced yes)
@@
 		)
 	)
-	(label "I2C_SDA"
+	(label "I2C_SCL"
 		(at 327.66 474.98 180)
 		(fields_autoplaced yes)
@@
 	)
 	(symbol
-		(lib_id "power:+3V3")
-		(at 327.66 480.06 90)
+		(lib_id "power:GND")
+		(at 327.66 480.06 270)
 		(unit 1)
 		(exclude_from_sim no)
@@
 			)
 		)
-		(property "Value" "+3V3"
+		(property "Value" "GND"
 			(at 330.2 485.14 0)
 			(effects
@@
 		)
 	)
-	(text "CONFIRM order: VCC GND SCK SDI SDO(=high, addr 0x77) CSB(=high, I2C)"
+	(text "order INT CS SDO SDI SCK VCC GND as on the module (checked 2026-09-29); CS high = I2C, SDO high = addr 0x77"
 		(exclude_from_sim no)
 		(at 353.06 472.44 0)
@@
 	)
 	(symbol
-		(lib_id "Connector_Generic:Conn_01x04")
-		(at 332.74 500.38 0)
+		(lib_id "Connector_Generic:Conn_01x05")
+		(at 332.74 505.46 0)
 		(unit 1)
 		(exclude_from_sim no)
@@
 		(dnp no)
 		(property "Reference" "J7"
-			(at 331.47 494.03 0)
+			(at 331.47 496.57 0)
 			(effects
 				(font
@@
 		)
 		(property "Value" "GPS MAX-M10S"
-			(at 339.09 501.65 0)
+			(at 339.09 506.73 0)
 			(effects
 				(font
@@
 			)
 		)
-		(property "Footprint" "Connector_PinSocket_2.54mm:PinSocket_1x04_P2.54mm_Vertical"
-			(at 332.74 500.38 0)
+		(property "Footprint" "Connector_PinSocket_2.54mm:PinSocket_1x05_P2.54mm_Vertical"
+			(at 332.74 505.46 0)
 			(effects
 				(font
@@
 		)
 		(property "Datasheet" ""
-			(at 332.74 500.38 0)
+			(at 332.74 505.46 0)
 			(effects
 				(font
@@
 		(pin "4"
 		)
+		(pin "5"
+		)
 		(instances
 			(project "hab1_flight"
@@
 	(symbol
 		(lib_id "power:+3V3")
-		(at 327.66 497.84 90)
+		(at 327.66 500.38 90)
 		(unit 1)
 		(exclude_from_sim no)
@@
 		(dnp no)
 		(property "Reference" "#PWR050"
-			(at 330.2 492.76 0)
+			(at 330.2 495.3 0)
 			(effects
 				(font
@@
 		)
 		(property "Value" "+3V3"
-			(at 330.2 502.92 0)
+			(at 330.2 505.46 0)
 			(effects
 				(font
@@
 		)
 		(property "Footprint" ""
-			(at 327.66 497.84 0)
+			(at 327.66 500.38 0)
 			(effects
 				(font
@@
 		)
 		(property "Datasheet" ""
-			(at 327.66 497.84 0)
+			(at 327.66 500.38 0)
 			(effects
 				(font
@@
 	(symbol
 		(lib_id "power:GND")
-		(at 327.66 500.38 270)
+		(at 327.66 502.92 270)
 		(unit 1)
 		(exclude_from_sim no)
@@
 		(dnp no)
 		(property "Reference" "#PWR051"
-			(at 330.2 495.3 0)
+			(at 330.2 497.84 0)
 			(effects
 				(font
@@
 		)
 		(property "Value" "GND"
-			(at 330.2 505.46 0)
+			(at 330.2 508 0)
 			(effects
 				(font
@@
 		)
 		(property "Footprint" ""
-			(at 327.66 500.38 0)
+			(at 327.66 502.92 0)
 			(effects
 				(font
@@
 		)
 		(property "Datasheet" ""
-			(at 327.66 500.38 0)
+			(at 327.66 502.92 0)
 			(effects
 				(font
@@
 	)
 	(label "USART1_RX"
-		(at 327.66 502.92 180)
+		(at 327.66 505.46 180)
 		(fields_autoplaced yes)
 		(effects
@@
 	)
 	(label "USART1_TX"
-		(at 327.66 505.46 180)
+		(at 327.66 508 180)
+		(fields_autoplaced yes)
+		(effects
+			(font
+				(size 1.27 1.27)
+			)
+			(justify right bottom)
+		)
+	)
+	(label "GPS_PPS"
+		(at 327.66 510.54 180)
 		(fields_autoplaced yes)
 		(effects
@@
 		)
 	)
-	(text "CONFIRM order: VCC GND TX(module) RX(module)"
+	(text "order VCC GND TX RX PPS as on the module (checked 2026-09-29); module TX -> MCU RX"
 		(exclude_from_sim no)
-		(at 353.06 500.38 0)
+		(at 353.06 505.46 0)
 		(effects
 			(font
@@
 	(symbol
 		(lib_id "Connector_Generic:Conn_01x03")
-		(at 332.74 528.32 0)
+		(at 332.74 533.4 0)
 		(unit 1)
 		(exclude_from_sim no)
@@
 		(dnp no)
 		(property "Reference" "J8"
-			(at 331.47 521.97 0)
+			(at 331.47 527.05 0)
 			(effects
 				(font
@@
 		)
 		(property "Value" "DS18B20 probe"
-			(at 339.09 529.59 0)
+			(at 339.09 534.67 0)
 			(effects
 				(font
@@
 		)
 		(property "Footprint" "Connector_JST:JST_XH_B3B-XH-A_1x03_P2.50mm_Vertical"
-			(at 332.74 528.32 0)
+			(at 332.74 533.4 0)
 			(effects
 				(font
@@
 		)
 		(property "Datasheet" ""
-			(at 332.74 528.32 0)
+			(at 332.74 533.4 0)
 			(effects
 				(font
@@
 	(symbol
 		(lib_id "power:+3V3")
-		(at 327.66 525.78 90)
+		(at 327.66 530.86 90)
 		(unit 1)
 		(exclude_from_sim no)
@@
 		(dnp no)
 		(property "Reference" "#PWR052"
-			(at 330.2 520.7 0)
+			(at 330.2 525.78 0)
 			(effects
 				(font
@@
 		)
 		(property "Value" "+3V3"
-			(at 330.2 530.86 0)
+			(at 330.2 535.94 0)
 			(effects
 				(font
@@
 		)
 		(property "Footprint" ""
-			(at 327.66 525.78 0)
+			(at 327.66 530.86 0)
 			(effects
 				(font
@@
 		)
 		(property "Datasheet" ""
-			(at 327.66 525.78 0)
+			(at 327.66 530.86 0)
 			(effects
 				(font
@@
 	)
 	(label "DS18B20_DQ"
-		(at 327.66 528.32 180)
+		(at 327.66 533.4 180)
 		(fields_autoplaced yes)
 		(effects
@@
 	(symbol
 		(lib_id "power:GND")
-		(at 327.66 530.86 270)
+		(at 327.66 535.94 270)
 		(unit 1)
 		(exclude_from_sim no)
@@
 		(dnp no)
 		(property "Reference" "#PWR053"
-			(at 330.2 525.78 0)
+			(at 330.2 530.86 0)
 			(effects
 				(font
@@
 		)
 		(property "Value" "GND"
-			(at 330.2 535.94 0)
+			(at 330.2 541.02 0)
 			(effects
 				(font
@@
 		)
 		(property "Footprint" ""
-			(at 327.66 530.86 0)
+			(at 327.66 535.94 0)
 			(effects
 				(font
@@
 		)
 		(property "Datasheet" ""
-			(at 327.66 530.86 0)
+			(at 327.66 535.94 0)
 			(effects
 				(font
@@
 	(text "red / yellow / black"
 		(exclude_from_sim no)
-		(at 353.06 528.32 0)
+		(at 353.06 533.4 0)
 		(effects
 			(font

Commit message: hardware: OLED socket order confirmed from the module (HW-24)
Co-Authored-By: Claude Opus 5.5 (1M context) <noreply@anthropic.com>
Claude-Session: https://claude.ai/code/session_01Y9WTd2yaDzj6r4py6E8uJo
Other:
- note added: "order GND VDD SCK SDA as on the module (checked 2026-09-29)"
- note removed: "CONFIRM order GND VCC SCL SDA"
Changed lines of the file:
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@@
 		)
 	)
-	(text "CONFIRM order GND VCC SCL SDA"
+	(text "order GND VDD SCK SDA as on the module (checked 2026-09-29)"
 		(exclude_from_sim no)
 		(at 431.8 137.16 0)

Commit message: hardware: recovery buzzer on PB4 (HW-24)
Active piezo buzzer on a 2-pin JST cable to the box wall, switched on the
low side by an AO3400A from the battery rail (loud), 100k gate pull-down so
it stays silent during boot, 1N4148W in case a magnetic buzzer is used.
ERC 0, netlist check 0 mismatches, PCB parity 0.

Co-Authored-By: Claude Opus 5.5 (1M context) <noreply@anthropic.com>
Claude-Session: https://claude.ai/code/session_01Y9WTd2yaDzj6r4py6E8uJo
Parts:
- added D3: 1N4148W, Diode_SMD:D_SOD-123, symbol Device:D
- added J11: BUZZER (+ / -), Connector_JST:JST_XH_B2B-XH-A_1x02_P2.50mm_Vertical, symbol Connector_Generic:Conn_01x02
- added Q2: AO3400A, Package_TO_SOT_SMD:SOT-23, symbol Transistor_FET:AO3400A
- added R12: 100k, Resistor_SMD:R_0603_1608Metric, symbol Device:R
Connections:
- net GND: now also Q2.2 (S), R12.2
- net VBAT_PROT: now also D3.1 (K), J11.1 (Pin_1)
- net BUZZER: now reaches U1.57 (PB4)
- net BUZZER: now also Q2.1 (G), R12.1
- new net BUZ_N: D3.2 (A), J11.2 (Pin_2), Q2.3 (D)
- no-connect marks 25 -> 24
Other:
- note added: "RECOVERY BUZZER battery rail, low-side FET"
- note added: "only needed if a magnetic buzzer is used"
- note added: "pin 1 = buzzer +, pin 2 = buzzer -"
- moved on the sheet: C14, H1, H2, H3, H4, J10, J4, J5, J6, J7, J8, J9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

Commit message: flight PCB: expansion header J12 (3V3, battery rail, 4 analog pins, 2 PWM pins), rerouted
ERC 0/0, netlist check 0 mismatches, DRC 0 unconnected, 0 parity issues.

Co-Authored-By: Claude Opus 5.5 (1M context) <noreply@anthropic.com>
Claude-Session: https://claude.ai/code/session_01Y9WTd2yaDzj6r4py6E8uJo
Parts:
- added J12: EXPANSION, Connector_PinSocket_2.54mm:PinSocket_1x10_P2.54mm_Vertical, symbol Connector_Generic:Conn_01x10
Connections:
- net +3V3: now also J12.1 (Pin_1)
- net GND: now also J12.10 (Pin_10), J12.2 (Pin_2)
- net VBAT_PROT: now also J12.3 (Pin_3)
- net EXP_A1: now reaches U1.13 (PA1)
- net EXP_A1: now also J12.4 (Pin_4)
- net EXP_A2: now reaches U1.18 (PA4)
- net EXP_A2: now also J12.5 (Pin_5)
- net EXP_PWM1: now reaches U1.58 (PB5)
- net EXP_PWM1: now also J12.8 (Pin_8)
- net EXP_PWM2: now reaches U1.60 (PB7)
- net EXP_PWM2: now also J12.9 (Pin_9)
- net EXP_A3: now reaches U1.8 (PC0)
- net EXP_A3: now also J12.6 (Pin_6)
- net EXP_A4: now reaches U1.9 (PC1)
- net EXP_A4: now also J12.7 (Pin_7)
- no-connect marks 24 -> 18
Other:
- note added: "A1..A4 = PA1 PA4 PC0 PC1 (ADC), PWM1/2 = PB5 PB7 (TIM3_CH2 / TIM4_CH2); pin 3 is the battery rail, NOT 3.3 V"
- moved on the sheet: H1, H2, H3, H4, TP1, TP10, TP2, TP3, TP4, TP5, TP6, TP7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

Commit message: flight PCB: fix swapped console TX/RX on the STDC14 connector, buzzer gate pull-down 4.7k; add the independent review report (HW-153)
Review finding B1: STDC14 pin 13 is the target RX (PA3), pin 14 the target TX (PA2).
ERC 0/0, netlist 0 mismatches, DRC 0 unconnected, 0 parity issues.

Co-Authored-By: Claude Opus 5.5 (1M context) <noreply@anthropic.com>
Claude-Session: https://claude.ai/code/session_01Y9WTd2yaDzj6r4py6E8uJo
Parts:
- R12: value 100k -> 4.7k
Connections:
- net VCP_RX: now also J3.13 (VCP_RX); no longer J3.14 (VCP_TX)
- net VCP_TX: now also J3.14 (VCP_TX); no longer J3.13 (VCP_RX)
Other:
- note added: "STDC14 names are target-centred (UM2448, UM2505 table 14): pin 13 T_VCP_RX = target RX (PA3), pin 14 T_VCP_TX = target TX (PA2)"
- note removed: "pin 13 VCP_RX (probe input) <- MCU TX; pin 14 VCP_TX -> MCU RX"
Changed lines of the file:
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@@
+		)
+	)
+	(label "VCP_RX"
+		(at 345.44 114.3 0)
+		(fields_autoplaced yes)
+		(effects
+			(font
+				(size 1.27 1.27)
+			)
+			(justify left bottom)
 		)
 	)
 	(label "VCP_TX"
-		(at 345.44 114.3 0)
-		(fields_autoplaced yes)
-		(effects
-			(font
-				(size 1.27 1.27)
-			)
-			(justify left bottom)
-		)
-	)
-	(label "VCP_RX"
 		(at 345.44 116.84 0)
 		(fields_autoplaced yes)
@@
 		)
 	)
-	(text "pin 13 VCP_RX (probe input) <- MCU TX; pin 14 VCP_TX -> MCU RX"
+	(text "STDC14 names are target-centred (UM2448, UM2505 table 14): pin 13 T_VCP_RX = target RX (PA3), pin 14 T_VCP_TX = target TX (PA2)"
 		(exclude_from_sim no)
 		(at 353.06 104.14 0)
@@
 			)
 		)
-		(property "Value" "100k"
+		(property "Value" "4.7k"
 			(at 330.2 420.37 0)
 			(effects

Commit message: flight PCB: review fixes - fuses, cable protection, SCL off the BOOT0 pin, decoupling at the pins, silkscreen pin names (HW-153)
F1/F2 resettable fuses, series resistors on the DS18B20 cable and the expansion
header, I2C SCL moved PB8 -> PA15 with PB8 pulled down, 100 nF 2 mm from each VDD
pin and at NRST / VDDA, pull-downs on LORA_TXEN/RXEN, module and pin names on silk.
ERC 0/0, netlist 0 mismatches, DRC 0 unconnected, 0 parity issues.

Co-Authored-By: Claude Opus 5.5 (1M context) <noreply@anthropic.com>
Claude-Session: https://claude.ai/code/session_01Y9WTd2yaDzj6r4py6E8uJo
Parts:
- added C15: 100n, Capacitor_SMD:C_0603_1608Metric, symbol Device:C
- added F1: PTC 0.5A hold, Fuse:Fuse_1206_3216Metric, symbol Device:Polyfuse
- added F2: PTC 0.2A hold, Fuse:Fuse_1206_3216Metric, symbol Device:Polyfuse
- added R13: 10k, Resistor_SMD:R_0603_1608Metric, symbol Device:R
- added R14, R15: 100, Resistor_SMD:R_0603_1608Metric, symbol Device:R
- added R16, R17, R18, R19, R20, R21: 1k, Resistor_SMD:R_0603_1608Metric, symbol Device:R
- added R22, R23: 100k, Resistor_SMD:R_0603_1608Metric, symbol Device:R
Connections:
- net +3V3: now also J12.3 (Pin_3), R14.1; no longer J12.1 (Pin_1), J8.1 (Pin_1)
- net DS18B20_DQ: now also R15.1; no longer J8.2 (Pin_2)
- net EXP_A1: now also R16.1; no longer J12.4 (Pin_4)
- net EXP_A2: now also R17.1; no longer J12.5 (Pin_5)
- net EXP_A3: now also R18.1; no longer J12.6 (Pin_6)
- net EXP_A4: now also R19.1; no longer J12.7 (Pin_7)
- net EXP_PWM1: now also R20.1; no longer J12.8 (Pin_8)
- net EXP_PWM2: now also R21.1; no longer J12.9 (Pin_9)
- net GND: now also C15.2, R13.2, R22.2, R23.2
- net I2C_SCL: now also U1.51 (PA15); no longer U1.61 (PB8)
- net LORA_RXEN: now also R23.1
- net LORA_TXEN: now also R22.1
- net NRST: now also C15.1
- net VBAT_PROT: now also J12.1 (Pin_1), F2.1; no longer D3.1 (K), J11.1 (Pin_1), J12.3 (Pin_3)
- net VBAT_RAW: now also F1.2; no longer J1.1 (Pin_1)
- new net BOOT0: R13.1, U1.61 (PB8)
- new net BUZ_P: D3.1 (K), F2.2, J11.1 (Pin_1)
- new net DS_DQ: J8.2 (Pin_2), R15.2
- new net DS_VCC: J8.1 (Pin_1), R14.2
- new net VBAT_IN: F1.1, J1.1 (Pin_1)
- new net X_A1: J12.4 (Pin_4), R16.2
- new net X_A2: J12.5 (Pin_5), R17.2
- new net X_A3: J12.6 (Pin_6), R18.2
- new net X_A4: J12.7 (Pin_7), R19.2
- new net X_PWM1: J12.8 (Pin_8), R20.2
- new net X_PWM2: J12.9 (Pin_9), R21.2
- no-connect marks 18 -> 17
Other:
- note added: "A1..A4 = PA1 PA4 PC0 PC1 (ADC), PWM1/2 = PB5 PB7 (TIM3_CH2 / TIM4_CH2), each through 1k; pin 1 is the battery rail, NOT 3.3 V (GND sits between it and the rest)"
- note removed: "A1..A4 = PA1 PA4 PC0 PC1 (ADC), PWM1/2 = PB5 PB7 (TIM3_CH2 / TIM4_CH2); pin 3 is the battery rail, NOT 3.3 V"
- moved on the sheet: C1, C10, C11, C12, C13, C14, C2, C3, C4, C5, C6, C7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
