File: hardware/flight_pcb/hab1_flight.kicad_sch (KiCad schematic)
At the start: 75 parts, among them J1 BATTERY 4xL91, J10 OLED SSD1306 (bench), J11 BUZZER (+ / -), J12 EXPANSION, J2 POWER SWITCH (on the box), J3 STDC14 SWD+VCP, J4 SPI FLASH module, J5 IMU GY-601N1, J6 BAROMETER BMP390, J7 GPS MAX-M10S, J8 DS18B20 probe, J9 LoRa E22-400M22S (adapter), Q1 AO3401A, Q2 AO3400A, SW1 RESET, U1 STM32G474RET6, U2 MIC5219-3.3

Commit message: flight PCB: regulator MIC5219 (SOT-23-5) -> LDL1117S33R (SOT-223), enough for LoRa TX current (HW-153)
ERC 0/0, netlist 0 mismatches, DRC 0 unconnected, 0 parity issues.
Pin order taken as the LD1117 symbol; to be confirmed against the datasheet before ordering.

Co-Authored-By: Claude Opus 5.5 (1M context) <noreply@anthropic.com>
Claude-Session: https://claude.ai/code/session_01Y9WTd2yaDzj6r4py6E8uJo
Parts:
- removed C3: 470p, Capacitor_SMD:C_0603_1608Metric, symbol Device:C
- C1: value 10u -> 10u 16V
- U2: value MIC5219-3.3 -> LDL1117S33R; footprint Package_TO_SOT_SMD:SOT-23-5 -> Package_TO_SOT_SMD:SOT-223-3_TabPin2; symbol Regulator_Linear:MIC5219-3.3YM5 -> Regulator_Linear:LD1117S33TR_SOT223
Connections:
- net +3V3: now also U2.2 (VO); no longer U2.5 (OUT)
- net GND: now also U2.1 (GND); no longer U2.2 (GND)
- net VBAT_PROT: no longer U2.1 (IN)
- removed net U2_BYP: U2.4 (BP)
Other:
- note added: "CONFIRM the pin order against the LDL1117 datasheet before ordering"
- note removed: "provisional, decide after HW-21"
- moved on the sheet: C1, C10, C11, C12, C13, C14, C15, C2, C4, C5, C6, C7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

Commit message: flight PCB: LDL1117 pinout confirmed from the datasheet; LoRa bulk capacitor 47u -> 4.7u to stay inside its stability chart (HW-153)
DS12022 rev 7: pins 1 GND, 2 VOUT, 3 VIN, tab VOUT; theta-JA 120 C/W; stability chart up to 22 uF.
ERC 0/0, netlist 0 mismatches, DRC 0 unconnected, 0 parity issues.

Co-Authored-By: Claude Opus 5.5 (1M context) <noreply@anthropic.com>
Claude-Session: https://claude.ai/code/session_01Y9WTd2yaDzj6r4py6E8uJo
Parts:
- C14: value 47u -> 4.7u; footprint Capacitor_SMD:C_1206_3216Metric -> Capacitor_SMD:C_0805_2012Metric
Other:
- note added: "pin order checked against DS12022 rev 7 table 1: 1 GND, 2 VOUT, 3 VIN, tab = VOUT"
- note removed: "CONFIRM the pin order against the LDL1117 datasheet before ordering"
Changed lines of the file:
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@@
 		)
 	)
-	(text "CONFIRM the pin order against the LDL1117 datasheet before ordering"
+	(text "pin order checked against DS12022 rev 7 table 1: 1 GND, 2 VOUT, 3 VIN, tab = VOUT"
 		(exclude_from_sim no)
 		(at 271.78 190.5 0)
@@
 			)
 		)
-		(property "Value" "47u"
+		(property "Value" "4.7u"
 			(at 408.94 374.65 0)
 			(effects
@@
 			)
 		)
-		(property "Footprint" "Capacitor_SMD:C_1206_3216Metric"
+		(property "Footprint" "Capacitor_SMD:C_0805_2012Metric"
 			(at 411.48 373.38 0)
 			(effects

Commit message: flight PCB: JLCPCB files (gerbers, BOM with LCSC numbers, CPL), parts checked in the JLCPCB catalogue (HW-155)
LEDs red/yellow instead of green/blue (out of stock and too dim from 3.3 V), battery
fuse in the 24 V version, keyed programming header, via copper ring 0.15 mm.
ERC 0/0, netlist 0 mismatches, DRC 0 unconnected, 0 parity issues.

Co-Authored-By: Claude Opus 5.5 (1M context) <noreply@anthropic.com>
Claude-Session: https://claude.ai/code/session_01Y9WTd2yaDzj6r4py6E8uJo
Parts:
- D1: value ALIVE green -> ALIVE red
- D2: value GPS FIX blue -> GPS FIX yellow
- F1: value PTC 0.5A hold -> PTC 0.5A 24V
- F2: value PTC 0.2A hold -> PTC 0.2A 24V
Changed lines of the file:
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@@
 			)
 		)
-		(property "Value" "PTC 0.5A hold"
+		(property "Value" "PTC 0.5A 24V"
 			(at 248.92 100.33 0)
 			(effects
@@
 			)
 		)
-		(property "Value" "ALIVE green"
+		(property "Value" "ALIVE red"
 			(at 340.36 407.67 0)
 			(effects
@@
 			)
 		)
-		(property "Value" "GPS FIX blue"
+		(property "Value" "GPS FIX yellow"
 			(at 340.36 450.85 0)
 			(effects
@@
 			)
 		)
-		(property "Value" "PTC 0.2A hold"
+		(property "Value" "PTC 0.2A 24V"
 			(at 408.94 67.31 0)
 			(effects

Commit message: flight PCB: LoRa module E22-400M22S soldered on by JLCPCB instead of an adapter socket (HW-162, HW-155)
Own footprint from the Ebyte drawing, checked against the labels on the real module;
no tracks or vias under the module; JLCPCB part C411291 in the BOM.
ERC 0/0, netlist 0 mismatches, DRC 0 unconnected, 0 parity issues.

Co-Authored-By: Claude Opus 5.5 (1M context) <noreply@anthropic.com>
Claude-Session: https://claude.ai/code/session_01Y9WTd2yaDzj6r4py6E8uJo
Parts:
- removed J9: LoRa E22-400M22S (adapter), Connector_PinSocket_2.54mm:PinSocket_1x12_P2.54mm_Vertical, symbol Connector_Generic:Conn_01x12
- added C16: 100n, Capacitor_SMD:C_0603_1608Metric, symbol Device:C
- added U3: E22-400M22S, hab1:E22-400M22S, symbol Connector_Generic:Conn_01x22
Connections:
- net +3V3: now also C16.1, U3.9 (Pin_9)
- net GND: now also C16.2, U3.1 (Pin_1), U3.10 (Pin_10), U3.11 (Pin_11), U3.12 (Pin_12), U3.2 (Pin_2), U3.20 (Pin_20), U3.22 (Pin_22), U3.3 (Pin_3), U3.4 (Pin_4), U3.5 (Pin_5)
- net LORA_BUSY: now also U3.14 (Pin_14)
- net LORA_DIO1: now also U3.13 (Pin_13)
- net LORA_NRST: now also U3.15 (Pin_15)
- net LORA_NSS: now also U3.19 (Pin_19)
- net LORA_RXEN: now also U3.6 (Pin_6)
- net LORA_TXEN: now also U3.7 (Pin_7)
- net SPI2_MISO: now also U3.16 (Pin_16)
- net SPI2_MOSI: now also U3.17 (Pin_17)
- net SPI2_SCK: now also U3.18 (Pin_18)
- no-connect marks 17 -> 19
Other:
- note added: "1-5 GND, 6 RXEN, 7 TXEN, 8 DIO2, 9 VCC, 10-12 GND, 13 DIO1, 14 BUSY, 15 NRST, 16 MISO, 17 MOSI, 18 SCK, 19 NSS, 20 GND, 21 ANT, 22 GND"
- note removed: "rev A: E22 on a header until HW-6 is done"
- moved on the sheet: C14, H1, H2, H3, H4, J10, J12, R16, R17, R18, R19, R20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
